File: Board Designs/V3-UV_Watch/Adafruit NeoPixel Ring 12.sch (EAGLE design)
At the start: 25 parts, among them U1 ATMEGA32U4-AU

Commit message: adding eagle files
Parts:
- removed C10, C12, C2, C3, C4, C6, C8, C9: (no value), rcl:C-EUC0603
- added IC1: VEML6070, we-sensor:VEML6070
Connections:
- net GND: no longer C10.2, C12.2, C2.2, C3.2, C4.2, C6.2, C8.2, C9.2
- net VDD: no longer C10.1, C12.1, C2.1, C3.1, C4.1, C6.1, C8.1, C9.1
Other:
- moved on the sheet: U1
Changed lines of the file:
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@@
 <part name="LED12" library="microbuilder" deviceset="WS28115050" device=""/>
 <part name="GND1" library="supply1" deviceset="GND" device=""/>
-<part name="C2" library="rcl" deviceset="C-EU" device="C0603"/>
-<part name="C3" library="rcl" deviceset="C-EU" device="C0603"/>
-<part name="C4" library="rcl" deviceset="C-EU" device="C0603"/>
-<part name="C6" library="rcl" deviceset="C-EU" device="C0603"/>
-<part name="C8" library="rcl" deviceset="C-EU" device="C0603"/>
-<part name="C9" library="rcl" deviceset="C-EU" device="C0603"/>
-<part name="C10" library="rcl" deviceset="C-EU" device="C0603"/>
-<part name="C12" library="rcl" deviceset="C-EU" device="C0603"/>
-<part name="GND2" library="supply1" deviceset="GND" device=""/>
 <part name="VDD1" library="supply1" deviceset="VDD" device=""/>
-<part name="VDD2" library="supply1" deviceset="VDD" device=""/>
 <part name="JP1" library="NeoPixelRing" deviceset="PINHD-1X1" device="CB"/>
 <part name="JP2" library="NeoPixelRing" deviceset="PINHD-1X1" device="CB"/>
@@
 <part name="JP4" library="NeoPixelRing" deviceset="PINHD-1X1" device="CB"/>
 <part name="U1" library="Microcontroller" library_urn="urn:adsk.eagle:library:11396388" deviceset="ATMEGA32U4-AU" device="" package3d_urn="urn:adsk.eagle:package:10882633/3"/>
+<part name="IC1" library="we-sensor" deviceset="VEML6070" device=""/>
 </parts>
 <sheets>
@@
 <attribute name="VALUE" x="358.14" y="58.42" size="1.778" layer="96"/>
 </instance>
-<instance part="C2" gate="G$1" x="63.5" y="129.54" smashed="yes">
-<attribute name="NAME" x="65.024" y="129.921" size="1.778" layer="95"/>
-<attribute name="VALUE" x="65.024" y="124.841" size="1.778" layer="96"/>
-</instance>
-<instance part="C3" gate="G$1" x="73.66" y="129.54" smashed="yes">
-<attribute name="NAME" x="75.184" y="129.921" size="1.778" layer="95"/>
-<attribute name="VALUE" x="75.184" y="124.841" size="1.778" layer="96"/>
-</instance>
-<instance part="C4" gate="G$1" x="83.82" y="129.54" smashed="yes">
-<attribute name="NAME" x="85.344" y="129.921" size="1.778" layer="95"/>
-<attribute name="VALUE" x="85.344" y="124.841" size="1.778" layer="96"/>
-</instance>
-<instance part="C6" gate="G$1" x="104.14" y="129.54" smashed="yes">
-<attribute name="NAME" x="105.664" y="129.921" size="1.778" layer="95"/>
-<attribute name="VALUE" x="105.664" y="124.841" size="1.778" layer="96"/>
-</instance>
-<instance part="C8" gate="G$1" x="124.46" y="129.54" smashed="yes">
-<attribute name="NAME" x="125.984" y="129.921" size="1.778" layer="95"/>
-<attribute name="VALUE" x="125.984" y="124.841" size="1.778" layer="96"/>
-</instance>
-<instance part="C9" gate="G$1" x="134.62" y="129.54" smashed="yes">
-<attribute name="NAME" x="136.144" y="129.921" size="1.778" layer="95"/>
-<attribute name="VALUE" x="136.144" y="124.841" size="1.778" layer="96"/>
-</instance>
-<instance part="C10" gate="G$1" x="144.78" y="129.54" smashed="yes">
-<attribute name="NAME" x="146.304" y="129.921" size="1.778" layer="95"/>
-<attribute name="VALUE" x="146.304" y="124.841" size="1.778" layer="96"/>
-</instance>
-<instance part="C12" gate="G$1" x="165.1" y="129.54" smashed="yes">
-<attribute name="NAME" x="166.624" y="129.921" size="1.778" layer="95"/>
-<attribute name="VALUE" x="166.624" y="124.841" size="1.778" layer="96"/>
-</instance>
-<instance part="GND2" gate="1" x="165.1" y="116.84" smashed="yes">
-<attribute name="VALUE" x="162.56" y="114.3" size="1.778" layer="96"/>
-</instance>
 <instance part="VDD1" gate="G$1" x="365.76" y="101.6" smashed="yes">
 <attribute name="VALUE" x="363.22" y="99.06" size="1.778" layer="96" rot="R90"/>
-</instance>
-<instance part="VDD2" gate="G$1" x="165.1" y="139.7" smashed="yes">
-<attribute name="VALUE" x="162.56" y="137.16" size="1.778" layer="96" rot="R90"/>
 </instance>
 <instance part="JP1" gate="G$1" x="30.48" y="76.2" smashed="yes" rot="R180">
@@
 <attribute name="VALUE" x="36.83" y="71.12" size="1.778" layer="96" rot="R180"/>
 </instance>
-<instance part="U1" gate="G$1" x="276.86" y="190.5" smashed="yes">
-<attribute name="NAME" x="236.22" y="220.98" size="6.4516" layer="95" ratio="10"/>
-<attribute name="VALUE" x="236.22" y="152.4" size="6.4516" layer="96" ratio="10"/>
+<instance part="U1" gate="G$1" x="144.78" y="200.66" smashed="yes">
+<attribute name="NAME" x="104.14" y="231.14" size="6.4516" layer="95" ratio="10"/>
+<attribute name="VALUE" x="104.14" y="162.56" size="6.4516" layer="96" ratio="10"/>
+</instance>
+<instance part="IC1" gate="IC" x="233.68" y="147.32" smashed="yes">
+<attribute name="NAME" x="226.06" y="154.94" size="1.778" layer="95" align="top-left"/>
+<attribute name="VALUE" x="226.06" y="137.16" size="1.778" layer="96"/>
 </instance>
 </instances>
@@
 <pinref part="JP4" gate="G$1" pin="1"/>
 <wire x1="33.02" y1="66.04" x2="53.34" y2="66.04" width="0.1524" layer="91"/>
-</segment>
-<segment>
-<pinref part="C12" gate="G$1" pin="2"/>
-<pinref part="GND2" gate="1" pin="GND"/>
-<wire x1="165.1" y1="124.46" x2="165.1" y2="121.92" width="0.1524" layer="91"/>
-<wire x1="165.1" y1="121.92" x2="165.1" y2="119.38" width="0.1524" layer="91"/>
-<pinref part="C10" gate="G$1" pin="2"/>
-<wire x1="165.1" y1="121.92" x2="144.78" y2="121.92" width="0.1524" layer="91"/>
-<wire x1="144.78" y1="121.92" x2="144.78" y2="124.46" width="0.1524" layer="91"/>
-<pinref part="C9" gate="G$1" pin="2"/>
-<wire x1="144.78" y1="121.92" x2="134.62" y2="121.92" width="0.1524" layer="91"/>
-<wire x1="134.62" y1="121.92" x2="134.62" y2="124.46" width="0.1524" layer="91"/>
-<pinref part="C8" gate="G$1" pin="2"/>
-<wire x1="134.62" y1="121.92" x2="124.46" y2="121.92" width="0.1524" layer="91"/>
-<wire x1="124.46" y1="121.92" x2="124.46" y2="124.46" width="0.1524" layer="91"/>
-<pinref part="C6" gate="G$1" pin="2"/>
-<wire x1="124.46" y1="121.92" x2="104.14" y2="121.92" width="0.1524" layer="91"/>
-<wire x1="104.14" y1="121.92" x2="104.14" y2="124.46" width="0.1524" layer="91"/>
-<pinref part="C4" gate="G$1" pin="2"/>
-<wire x1="104.14" y1="121.92" x2="83.82" y2="121.92" width="0.1524" layer="91"/>
-<wire x1="83.82" y1="121.92" x2="83.82" y2="124.46" width="0.1524" layer="91"/>
-<pinref part="C3" gate="G$1" pin="2"/>
-<wire x1="83.82" y1="121.92" x2="73.66" y2="121.92" width="0.1524" layer="91"/>
-<wire x1="73.66" y1="121.92" x2="73.66" y2="124.46" width="0.1524" layer="91"/>
-<pinref part="C2" gate="G$1" pin="2"/>
-<wire x1="73.66" y1="121.92" x2="63.5" y2="121.92" width="0.1524" layer="91"/>
-<wire x1="63.5" y1="121.92" x2="63.5" y2="124.46" width="0.1524" layer="91"/>
 </segment>
 </net>
@@
 <wire x1="33.02" y1="96.52" x2="50.8" y2="96.52" width="0.1524" layer="91"/>
 </segment>
-<segment>
-<pinref part="C12" gate="G$1" pin="1"/>
-<pinref part="VDD2" gate="G$1" pin="VDD"/>
-<wire x1="165.1" y1="132.08" x2="165.1" y2="134.62" width="0.1524" layer="91"/>
-<wire x1="165.1" y1="134.62" x2="165.1" y2="137.16" width="0.1524" layer="91"/>
-<wire x1="165.1" y1="134.62" x2="144.78" y2="134.62" width="0.1524" layer="91"/>
-<wire x1="144.78" y1="134.62" x2="134.62" y2="134.62" width="0.1524" layer="91"/>
-<wire x1="134.62" y1="134.62" x2="124.46" y2="134.62" width="0.1524" layer="91"/>
-<wire x1="124.46" y1="134.62" x2="104.14" y2="134.62" width="0.1524" layer="91"/>
-<wire x1="104.14" y1="134.62" x2="83.82" y2="134.62" width="0.1524" layer="91"/>
-<wire x1="83.82" y1="134.62" x2="73.66" y2="134.62" width="0.1524" layer="91"/>
-<wire x1="73.66" y1="134.62" x2="63.5" y2="134.62" width="0.1524" layer="91"/>
-<pinref part="C2" gate="G$1" pin="1"/>
-<wire x1="63.5" y1="132.08" x2="63.5" y2="134.62" width="0.1524" layer="91"/>
-<pinref part="C3" gate="G$1" pin="1"/>
-<wire x1="73.66" y1="132.08" x2="73.66" y2="134.62" width="0.1524" layer="91"/>
-<pinref part="C4" gate="G$1" pin="1"/>
-<wire x1="83.82" y1="132.08" x2="83.82" y2="134.62" width="0.1524" layer="91"/>
-<pinref part="C6" gate="G$1" pin="1"/>
-<wire x1="104.14" y1="132.08" x2="104.14" y2="134.62" width="0.1524" layer="91"/>
-<pinref part="C8" gate="G$1" pin="1"/>
-<wire x1="124.46" y1="132.08" x2="124.46" y2="134.62" width="0.1524" layer="91"/>
-<pinref part="C9" gate="G$1" pin="1"/>
-<wire x1="134.62" y1="132.08" x2="134.62" y2="134.62" width="0.1524" layer="91"/>
-<pinref part="C10" gate="G$1" pin="1"/>
-<wire x1="144.78" y1="132.08" x2="144.78" y2="134.62" width="0.1524" layer="91"/>
-</segment>
-</net>
+</net>
