File: Board Designs/V4-UV_Watch/V4-UV_Watch.brd (EAGLE design)
At the start: 36.8 x 36.8 mm, 21 parts, among them IC1 VEML6070, U1 ATMEGA32U4-AU

Commit message: V4 hardware
Parts:
- removed IC1: VEML6070, we-sensor:OPLGA
- added C10, C12, C2, C3, C4, C6, C8, C9: (no value), rcl:C0603
- added TP1, TP2, TP3, TP4: TESTPAD_TPSQTP20SQ, BeagleBone_Blue_R3:TESTPAD_TP20SQ
- added U2: ATMEGA32U4-AU, Microcontroller:44-TQFP
- U1: value ATMEGA32U4-AU -> VEML6070; device Microcontroller:44-TQFP -> VEML6070:PHODET_VEML6070
- moved JP4 1.42 mm to (32.5, 7.48)
- moved LED1 1.42 mm to (20.3, 34.4)
- moved LED4 1.42 mm to (35.1, 19.7)
- moved LED8 1.42 mm to (13.0, 6.93)
- moved JP3 1.42 mm to (15.9, 3.04)
- moved LED9 1.42 mm to (7.56, 12.3)
- moved LED12 1.42 mm to (13.0, 32.4)
- moved U$3 1.42 mm to (18.4, 31.8)
- moved LED6 1.42 mm to (27.7, 6.93)
- moved LED7 1.42 mm to (20.3, 4.95)
- moved JP2 1.42 mm to (8.12, 31.9)
- moved LED10 1.42 mm to (5.59, 19.7)
- moved LED11 1.42 mm to (7.56, 27.1)
- moved JP1 1.42 mm to (24.8, 36.3)
- moved LED2 1.42 mm to (27.7, 32.4)
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Connections:
- removed net VCC: IC1.6
- net AVCC_24: now also U2.24; no longer U1.24
- net AVCC_44: now also U2.44; no longer U1.44
- net GND: now also C10.2, C12.2, C2.2, C3.2, C4.2, C6.2, C8.2, C9.2, U1.1; no longer IC1.1
- net GND_15: now also U2.15; no longer U1.15
- net GND_23: now also U2.23; no longer U1.23
- net GND_35: now also U2.35; no longer U1.35
- net GND_43: now also U2.43; no longer U1.43
- net UCAP: now also U2.6; no longer U1.6
- net UGND: now also U2.5; no longer U1.5
- net UVCC: now also U2.2; no longer U1.2
- net VCC_14: now also U2.14; no longer U1.14
- net VCC_34: now also U2.34; no longer U1.34
- net VDD: now also C10.1, C12.1, C2.1, C3.1, C4.1, C6.1, C8.1, C9.1, U1.6
Routing:
- net VDD: track 155.5 -> 159.6 mm, vias 13 -> 12
Other:
- outline, holes or cut-outs redrawn
